File: Power/kill_control/kill_control.kicad_sch (KiCad schematic)
At the start: 74 parts, among them J1 Debug, J4 t, U2 AMS1117-3.3, U3 TPS5430DDA, Y1 12MHz*

Commit message: add pdf
Other:
- note removed: "все приходится делать самому"
Changed lines of the file:
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@@
-    (effects (font (size 1.27 1.27)) (justify left bottom))
-  )
-  (text "все приходится делать самому" (at 252.73 190.5 0)
     (effects (font (size 1.27 1.27)) (justify left bottom))
   )
