File: Power/psu2psu01/psu2psu01.kicad_sch (KiCad schematic)
At the start: 137 parts, among them J1 CONN01PIN, J2 CONN01PIN, J3 CONN01PIN, J4 CONN01PIN, J5 CONN01PIN, J6 CONN01PIN, T1 HM1243, T2 YC13006, T3 HB13006, U1 DM311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

Commit message: up
Parts:
- removed C38: 470x63, mmods:CP4, symbol _aa40_capacitors:C_CAP_PLUS
- removed C41: 0,1, Capacitor_SMD:C_1206_3216Metric, symbol _aa40_capacitors:C_CAP
- removed R27: *, ma_misc:RSHUNT1, symbol _aa40_resistors:R_SHUNT
- removed R53, R54, R55, R56, R57, R58, R59, R60, R61, R62, R63, R64, R65: 10, Resistor_SMD:R_1206_3216Metric, symbol _aa40_resistors:R_RES_0.125W
- added R40, R41, R42: 47, mmods:RES2WV01, symbol _aa40_resistors:R_RES_2.0W
- added R43, R44, R45, R46, R47, R48, R49, R50: ~, Resistor_SMD:R_1206_3216Metric, symbol _aa40_resistors:R_RES_0.125W
- C25: value 0,01 -> 0,033
- C27, C30: footprint mmods:CP4 -> Capacitor_THT:CP_Radial_D14.0mm_P5.00mm
- C36, C37: footprint Capacitor_SMD:C_1206_3216Metric -> Capacitor_THT:C_Disc_D3.0mm_W2.0mm_P2.50mm
- D16, D17: footprint Package_TO_SOT_THT:TO-3P-3_Vertical -> mmods:TO-220-3-01
- R24: value 2k4 -> 1k2
- R25: value 82 -> 75; footprint Capacitor_SMD:C_1206_3216Metric -> Resistor_THT:R_Axial_DIN0207_L6.3mm_D2.5mm_P10.16mm_Horizontal
- R30: value 33k -> 120k*
- R31: value 1k -> 10k
- R33: value 500 -> 5k
- R34: value 4k7 -> 10k
- R38: value 33k -> 47k*
- R51, R52: value 10 -> ~
Connections:
- net GND: now also C28.2, R51.2, R52.2, R43.2, R44.2, R45.2, R46.2, R47.2, R48.2, R49.2, R50.2
- net GND0: now also R51.1, R52.1, R42.1, R43.1, R44.1, R45.1, R46.1, R47.1, R48.1, R49.1, R50.1; no longer C28.2
- net at D16.1 (A1), D16.3 (A2), T3.6: now also R40.2; no longer C37.2
- net at D16.2 (K), D17.2 (K), L2.1: now also C37.2, R41.2; no longer R51.1, R52.1
- net at C27.1, C28.1, C30.1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: now also R42.2
- net at C37.1: now also R40.1
- new net: C36.2, R41.1
Other:
- note added: "5 ... 36 вольт"
- note added: "D14P5"
- note removed: "10k"
- note removed: "1k2"
- note removed: "27k"
- note removed: "5k???"
- note removed: "D12.5P5"
- moved on the sheet: C31, C37

Commit message: up
Parts:
- R30: value 120k* -> 100k*
Other:
- note removed: "4k7"
- moved on the sheet: D18, R66
Changed lines of the file:
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@@
   (junction (at 69.215 120.015) (diameter 0) (color 0 0 0 0)
   )
-  (junction (at 127.635 49.53) (diameter 0) (color 0 0 0 0)
-  )
   (junction (at 151.765 99.06) (diameter 0) (color 0 0 0 0)
   )
@@
   (junction (at 60.96 22.86) (diameter 0) (color 0 0 0 0)
   )
+  (junction (at 127.635 50.8) (diameter 0) (color 0 0 0 0)
+  )
   (wire (pts (xy 212.09 78.74) (xy 210.82 78.74))
     (stroke (width 0) (type default))
@@
     (stroke (width 0) (type default))
   )
+  (wire (pts (xy 127.635 50.8) (xy 127.635 57.15))
+    (stroke (width 0) (type default))
+  )
   (wire (pts (xy 214.63 126.365) (xy 214.63 130.175))
     (stroke (width 0) (type default))
@@
     (stroke (width 0) (type default))
   )
-  (wire (pts (xy 127.635 46.355) (xy 127.635 49.53))
-    (stroke (width 0) (type default))
-  )
   (wire (pts (xy 87.63 155.575) (xy 118.11 155.575))
     (stroke (width 0) (type default))
@@
     (stroke (width 0) (type default))
   )
-  (wire (pts (xy 127.635 49.53) (xy 128.905 49.53))
+  (wire (pts (xy 127.635 50.8) (xy 128.905 50.8))
     (stroke (width 0) (type default))
   )
@@
     (stroke (width 0) (type default))
   )
-  (wire (pts (xy 139.065 49.53) (xy 140.335 49.53))
+  (wire (pts (xy 139.065 50.8) (xy 140.335 50.8))
     (stroke (width 0) (type default))
   )
@@
     (stroke (width 0) (type default))
   )
-  (wire (pts (xy 127.635 49.53) (xy 127.635 57.15))
+  (wire (pts (xy 127.635 46.355) (xy 127.635 50.8))
     (stroke (width 0) (type default))
   )
@@
     (stroke (width 0) (type default))
   )
-  (wire (pts (xy 147.955 49.53) (xy 149.86 49.53))
+  (wire (pts (xy 147.955 50.8) (xy 149.86 50.8))
     (stroke (width 0) (type default))
   )
@@
     (effects (font (size 1.27 1.27) italic) (justify right bottom))
   )
-  (text "4k7" (at 65.405 133.35 0)
-    (effects (font (size 1.27 1.27)) (justify left bottom))
-  )
   (text "+" (at 75.565 115.57 0)
     (effects (font (size 1.27 1.27)) (justify left bottom))
@@
     (effects (font (size 1.27 1.27) italic) (justify left bottom))
   )
-  (global_label "P4" (shape input) (at 117.475 123.19 90) (fields_autoplaced)
-    (effects (font (size 1.27 1.27)) (justify left))
-    (property "Intersheetrefs" "${INTERSHEET_REFS}" (at 117.475 117.7253 90)
-      (effects (font (size 1.27 1.27)) (justify left) hide)
-    )
-  )
   (global_label "Stb" (shape input) (at 127.635 46.355 90) (fields_autoplaced)
     (effects (font (size 1.27 1.27)) (justify left))
@@
       (effects (font (size 1.016 1.016)))
     )
-    (property "Value" "120k*" (at 40.64 140.335 0)
+    (property "Value" "100k*" (at 40.64 140.335 0)
       (effects (font (size 1.016 1.016)))
     )
@@
     )
   )
-  (symbol (lib_id "_aa40_resistors:R_RES_0.125W") (at 133.985 49.53 0) (mirror y) (unit 1)
+  (symbol (lib_id "_aa40_resistors:R_RES_0.125W") (at 133.985 50.8 0) (mirror y) (unit 1)
     (in_bom yes) (on_board yes) (dnp no)
-    (property "Reference" "R66" (at 133.985 46.99 0)
+    (property "Reference" "R66" (at 133.985 48.26 0)
       (effects (font (size 1.016 1.016)))
     )
-    (property "Value" "10" (at 133.985 52.07 0)
+    (property "Value" "10" (at 133.985 53.34 0)
       (effects (font (size 1.016 1.016)) hide)
     )
-    (property "Footprint" "Resistor_SMD:R_1206_3216Metric" (at 137.795 52.07 0)
+    (property "Footprint" "Resistor_SMD:R_1206_3216Metric" (at 137.795 53.34 0)
       (effects (font (size 1.778 1.778)) hide)
     )
-    (property "Datasheet" "" (at 133.985 49.53 0)
+    (property "Datasheet" "" (at 133.985 50.8 0)
       (effects (font (size 1.778 1.778)) hide)
     )
@@
     )
   )
-  (symbol (lib_id "_aa40_misc:GND") (at 151.13 49.53 90) (unit 1)
+  (symbol (lib_id "_aa40_misc:GND") (at 151.13 50.8 90) (unit 1)
     (in_bom yes) (on_board yes) (dnp no)
-    (property "Reference" "#PWR017" (at 152.4 49.53 0)
+    (property "Reference" "#PWR017" (at 152.4 50.8 0)
       (effects (font (size 1.016 1.016)) hide)
     )
-    (property "Value" "GND" (at 152.4 49.53 0)
+    (property "Value" "GND" (at 152.4 50.8 0)
       (effects (font (size 1.016 1.016)) hide)
     )
-    (property "Footprint" "" (at 151.13 49.53 0)
+    (property "Footprint" "" (at 151.13 50.8 0)
       (effects (font (size 1.27 1.27)) hide)
     )
-    (property "Datasheet" "" (at 151.13 49.53 0)
+    (property "Datasheet" "" (at 151.13 50.8 0)
       (effects (font (size 1.27 1.27)) hide)
     )
@@
   (symbol (lib_id "_aa40_misc:CONN01PIN") (at 134.62 57.15 0) (unit 1)
     (in_bom yes) (on_board yes) (dnp no)
-    (property "Reference" "J3" (at 134.62 54.61 0)
+    (property "Reference" "J3" (at 134.62 55.88 0)
       (effects (font (size 1.016 1.016)))
     )
@@
     )
   )
-  (symbol (lib_id "_aa40_diodes:LED2") (at 144.145 49.53 90) (unit 1)
+  (symbol (lib_id "_aa40_diodes:LED2") (at 144.145 50.8 90) (unit 1)
     (in_bom yes) (on_board yes) (dnp no)
-    (property "Reference" "D18" (at 144.145 45.085 90)
+    (property "Reference" "D18" (at 144.145 46.355 90)
       (effects (font (size 1.016 1.016)))
     )
-    (property "Value" "LED" (at 141.605 55.88 0)
+    (property "Value" "LED" (at 141.605 57.15 0)
       (effects (font (size 1.016 1.016)) (justify left) hide)
     )
-    (property "Footprint" "LED_SMD:LED_1206_3216Metric_ReverseMount_Hole1.8x2.4mm" (at 131.445 49.53 0)
+    (property "Footprint" "LED_SMD:LED_1206_3216Metric_ReverseMount_Hole1.8x2.4mm" (at 131.445 50.8 0)
       (effects (font (size 1.778 1.778)) hide)
     )
-    (property "Datasheet" "" (at 131.445 49.53 0)
+    (property "Datasheet" "" (at 131.445 50.8 0)
       (effects (font (size 1.778 1.778)) hide)
     )

Commit message: up
Parts:
- C11, C12: footprint mmods:CPD11mmW5mmP10mm01 -> mmods:CPD01
Changed lines of the file:
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@@
       (effects (font (size 1.016 1.016)))
     )
-    (property "Footprint" "mmods:CPD11mmW5mmP10mm01" (at 101.6 38.1 0)
+    (property "Footprint" "mmods:CPD01" (at 101.6 38.1 0)
       (effects (font (size 1.778 1.778)) hide)
     )
@@
       (effects (font (size 1.016 1.016)))
     )
-    (property "Footprint" "mmods:CPD11mmW5mmP10mm01" (at 101.6 27.94 0)
-      (effects (font (size 1.778 1.778)) hide)
-    )
+    (property "Footprint" "mmods:CPD01" (at 101.6 27.94 0)
+      (effects (font (size 1.778 1.778)) hide)
+    )

Commit message: up
Parts:
- D13: footprint Diode_SMD:D_1206_3216Metric -> Diode_SMD:D_SMA
Changed lines of the file:
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@@
       (effects (font (size 1.016 1.016)))
     )
-    (property "Footprint" "Diode_SMD:D_1206_3216Metric" (at 64.77 82.55 0)
+    (property "Footprint" "Diode_SMD:D_SMA" (at 64.77 82.55 0)
       (effects (font (size 1.778 1.778)) hide)
     )

Commit message: 30.01up
Parts:
- added R27: 15k, Capacitor_SMD:C_1206_3216Metric, symbol _aa40_resistors:R_RES_0.125W
- added R53: 33k, Capacitor_SMD:C_1206_3216Metric, symbol _aa40_resistors:R_RES_0.125W
- added VT5: BC807, Package_TO_SOT_SMD:SOT-23, symbol _aa40_transistors:BC807-40
Connections:
- net at C23.2, R31.1, R35.1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: now also R27.2, VT5.2 (E)
- net P4: no longer names the net of C23.1, R21.2, U4.4 (DTC)
- net P4: now also VT5.3 (C)
- new net: R27.1, R53.1, VT5.1 (B)
- new net SH: R53.2
Changed lines of the file:
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@@
   (junction (at 214.63 118.745) (diameter 0) (color 0 0 0 0)
   )
-  (junction (at 224.79 122.555) (diameter 0) (color 0 0 0 0)
+  (junction (at 44.45 106.045) (diameter 0) (color 0 0 0 0)
   )
-  (junction (at 69.215 120.015) (diameter 0) (color 0 0 0 0)
+  (junction (at 224.79 122.555) (diameter 0) (color 0 0 0 0)
   )
   (junction (at 151.765 99.06) (diameter 0) (color 0 0 0 0)
@@
   (junction (at 224.79 153.035) (diameter 0) (color 0 0 0 0)
   )
+  (junction (at 68.58 120.015) (diameter 0) (color 0 0 0 0)
+  )
   (junction (at 90.17 57.15) (diameter 0) (color 0 0 0 0)
   )
@@
   (junction (at 34.925 120.015) (diameter 0) (color 0 0 0 0)
   )
+  (junction (at 68.58 106.045) (diameter 0) (color 0 0 0 0)
+  )
   (junction (at 110.49 33.02) (diameter 0) (color 0 0 0 0)
   )
@@
   (junction (at 55.245 120.015) (diameter 0) (color 0 0 0 0)
   )
+  (junction (at 58.42 113.03) (diameter 0) (color 0 0 0 0)
+  )
   (junction (at 90.17 93.98) (diameter 0) (color 0 0 0 0)
   )
@@
     (stroke (width 0) (type default))
   )
-  (wire (pts (xy 69.215 116.84) (xy 69.215 120.015))
-    (stroke (width 0) (type default))
-  )
   (wire (pts (xy 214.63 137.795) (xy 214.63 141.605))
     (stroke (width 0) (type default))
@@
     (stroke (width 0) (type default))
   )
-  (wire (pts (xy 29.21 106.045) (xy 74.93 106.045))
+  (wire (pts (xy 29.21 106.045) (xy 44.45 106.045))
     (stroke (width 0) (type default))
   )
@@
     (stroke (width 0) (type default))
   )
+  (wire (pts (xy 68.58 106.045) (xy 74.93 106.045))
+    (stroke (width 0) (type default))
+  )
   (wire (pts (xy 242.57 99.06) (xy 257.81 99.06))
     (stroke (width 0) (type default))
@@
     (stroke (width 0) (type default))
   )
+  (wire (pts (xy 58.42 113.03) (xy 57.15 113.03))
+    (stroke (width 0) (type default))
+  )
   (wire (pts (xy 133.985 114.3) (xy 128.905 114.3))
     (stroke (width 0) (type default))
@@
     (stroke (width 0) (type default))
   )
+  (wire (pts (xy 58.42 113.03) (xy 62.23 113.03))
+    (stroke (width 0) (type default))
+  )
   (wire (pts (xy 133.985 86.36) (xy 133.985 88.9))
     (stroke (width 0) (type default))
   )
+  (wire (pts (xy 58.42 108.585) (xy 58.42 113.03))
+    (stroke (width 0) (type default))
+  )
   (wire (pts (xy 39.37 133.985) (xy 38.1 133.985))
     (stroke (width 0) (type default))
@@
     (stroke (width 0) (type default))
   )
-  (wire (pts (xy 67.31 120.015) (xy 69.215 120.015))
+  (wire (pts (xy 67.31 120.015) (xy 68.58 120.015))
     (stroke (width 0) (type default))
   )
@@
     (stroke (width 0) (type default))
   )
+  (wire (pts (xy 68.58 106.045) (xy 68.58 107.95))
+    (stroke (width 0) (type default))
+  )
   (wire (pts (xy 210.185 118.745) (xy 210.185 123.19))
     (stroke (width 0) (type default))
@@
     (stroke (width 0) (type default))
   )
+  (wire (pts (xy 44.45 113.03) (xy 46.99 113.03))
+    (stroke (width 0) (type default))
+  )
   (wire (pts (xy 87.63 155.575) (xy 118.11 155.575))
     (stroke (width 0) (type default))
@@
     (stroke (width 0) (type default))
   )
-  (wire (pts (xy 69.215 120.015) (xy 74.93 120.015))
-    (stroke (width 0) (type default))
-  )
   (wire (pts (xy 185.42 88.9) (xy 185.42 99.06))
     (stroke (width 0) (type default))
@@
     (stroke (width 0) (type default))
   )
+  (wire (pts (xy 46.99 108.585) (xy 44.45 108.585))
+    (stroke (width 0) (type default))
+  )
   (wire (pts (xy 139.065 50.8) (xy 140.335 50.8))
     (stroke (width 0) (type default))
@@
     (stroke (width 0) (type default))
   )
+  (wire (pts (xy 68.58 120.015) (xy 74.93 120.015))
+    (stroke (width 0) (type default))
+  )
   (wire (pts (xy 101.6 93.98) (xy 90.17 93.98))
     (stroke (width 0) (type default))
@@
     (stroke (width 0) (type default))
   )
+  (wire (pts (xy 58.42 108.585) (xy 57.15 108.585))
+    (stroke (width 0) (type default))
+  )
   (wire (pts (xy 87.63 43.18) (xy 69.85 43.18))
     (stroke (width 0) (type default))
@@
     (stroke (width 0) (type default))
   )
+  (wire (pts (xy 44.45 108.585) (xy 44.45 106.045))
+    (stroke (width 0) (type default))
+  )
   (wire (pts (xy 147.955 50.8) (xy 149.86 50.8))
     (stroke (width 0) (type default))
@@
     (stroke (width 0) (type default))
   )
+  (wire (pts (xy 68.58 118.11) (xy 68.58 120.015))
+    (stroke (width 0) (type default))
+  )
   (wire (pts (xy 110.49 40.64) (xy 110.49 44.45))
     (stroke (width 0) (type default))
@@
     (stroke (width 0) (type default))
   )
+  (wire (pts (xy 44.45 106.045) (xy 68.58 106.045))
+    (stroke (width 0) (type default))
+  )
   (wire (pts (xy 35.56 59.69) (xy 35.56 57.15))
     (stroke (width 0) (type default))
@@
     (effects (font (size 1.27 1.27) italic) (justify left bottom))
   )
-  (text "5 ... 36 вольт" (at 37.465 109.22 0)
+  (text "5 ... 36 вольт" (at 16.51 104.775 0)
     (effects (font (size 1.27 1.27)) (justify left bottom))
   )
@@
     )
   )
-  (global_label "P4" (shape input) (at 69.215 116.84 90) (fields_autoplaced)
-    (effects (font (size 1.27 1.27)) (justify left))
-    (property "Intersheetrefs" "${INTERSHEET_REFS}" (at 69.215 111.3753 90)
-      (effects (font (size 1.27 1.27)) (justify left) hide)
+  (global_label "SH" (shape input) (at 44.45 113.03 180) (fields_autoplaced)
+    (effects (font (size 1.27 1.27)) (justify right))
+    (property "Intersheetrefs" "${INTERSHEET_REFS}" (at 38.9248 113.03 0)
+      (effects (font (size 1.27 1.27)) (justify right) hide)
     )
   )
@@
     )
   )
+  (symbol (lib_id "_aa40_resistors:R_RES_0.125W") (at 52.07 113.03 0) (mirror y) (unit 1)
+    (in_bom yes) (on_board yes) (dnp no)
+    (property "Reference" "R53" (at 45.72 111.76 0)
+      (effects (font (size 1.016 1.016)) (justify right))
+    )
+    (property "Value" "33k" (at 54.61 111.76 0)
+      (effects (font (size 1.016 1.016)) (justify right))
+    )
+    (property "Footprint" "Capacitor_SMD:C_1206_3216Metric" (at 55.88 115.57 0)
+      (effects (font (size 1.778 1.778)) hide)
+    )
+    (property "Datasheet" "" (at 52.07 113.03 0)
+      (effects (font (size 1.778 1.778)) hide)
+    )
+    (pin "1")
+    (pin "2")
+    (instances
+      (project "psu2psu01"
+        (path "/f6d8bfcb-7ecc-4a03-a161-d509594d410b"
+          (reference "R53") (unit 1)
+        )
+      )
+    )
+  )
   (symbol (lib_id "_aa40_capacitors:C_CAP") (at 192.405 91.44 90) (unit 1)
     (in_bom yes) (on_board yes) (dnp no)
@@
     )
   )
+  (symbol (lib_id "_aa40_resistors:R_RES_0.125W") (at 52.07 108.585 0) (mirror y) (unit 1)
+    (in_bom yes) (on_board yes) (dnp no)
+    (property "Reference" "R27" (at 45.72 107.315 0)
+      (effects (font (size 1.016 1.016)) (justify right))
+    )
+    (property "Value" "15k" (at 54.61 107.315 0)
+      (effects (font (size 1.016 1.016)) (justify right))
+    )
+    (property "Footprint" "Capacitor_SMD:C_1206_3216Metric" (at 55.88 111.125 0)
+      (effects (font (size 1.778 1.778)) hide)
+    )
+    (property "Datasheet" "" (at 52.07 108.585 0)
+      (effects (font (size 1.778 1.778)) hide)
+    )
+    (pin "1")
+    (pin "2")
+    (instances
+      (project "psu2psu01"
+        (path "/f6d8bfcb-7ecc-4a03-a161-d509594d410b"
+          (reference "R27") (unit 1)
+        )
+      )
+    )
+  )
   (symbol (lib_id "_aa40_misc:GND") (at 262.89 96.52 0) (unit 1)
     (in_bom yes) (on_board yes) (dnp no)
@@
   (symbol (lib_id "_aa40_misc:CONN01PIN") (at 134.62 57.15 0) (unit 1)
     (in_bom yes) (on_board yes) (dnp no)
-    (property "Reference" "J3" (at 134.62 55.88 0)
+    (property "Reference" "J3" (at 134.62 54.61 0)
       (effects (font (size 1.016 1.016)))
     )
@@
         )
       )
+    )
+  )
+  (symbol (lib_id "_aa40_transistors:BC807-40") (at 67.31 113.03 0) (mirror x) (unit 1)
+    (in_bom yes) (on_board yes) (dnp no)
+    (property "Reference" "VT5" (at 59.055 108.585 0)
+      (effects (font (size 1.016 1.016)) (justify left))
+    )
+    (property "Value" "BC807" (at 59.055 110.49 0)
+      (effects (font (size 1.016 1.016)) (justify left))
+    )
+    (property "Footprint" "Package_TO_SOT_SMD:SOT-23" (at 67.1068 87.63 0)
+      (effects (font (size 1.778 1.778)) hide)
+    )
+    (property "Datasheet" "" (at 67.1068 87.63 0)
+      (effects (font (size 1.778 1.778)) hide)
+    )
+    (pin "1")
+    (pin "3")
+    (pin "2")
+    (instances
+      (project "psu2psu01"
+        (path "/f6d8bfcb-7ecc-4a03-a161-d509594d410b"
+          (reference "VT5") (unit 1)
+        )
+      )

Commit message: up
Parts:
- removed R43, R44, R45, R46, R47, R48, R49, R50, R51, R52: ~, Resistor_SMD:R_1206_3216Metric, symbol _aa40_resistors:R_RES_0.125W
- added R43, R44, R45: 0,1, Resistor_SMD:R_2512_6332Metric, symbol _aa40_resistors:R_RES_2.0W
- added R46: 3k*, mmods:RES2WV01, symbol _aa40_resistors:R_RES_2.0W
- added R47: 100*, Potentiometer_THT:Potentiometer_Bourns_3296W_Vertical, symbol _aa40_resistors:RP_TRIMMER
- R25: value 75 -> 10*; footprint Resistor_THT:R_Axial_DIN0207_L6.3mm_D2.5mm_P10.16mm_Horizontal -> Capacitor_SMD:C_1206_3216Metric
- R42: value 47 -> 3k*
Connections:
- net GND: now also R43.1, R44.1, R45.1; no longer H2.1
- net GND0: now also R43.2, R44.2, R45.2, R46.2, R47.2, R47.3; no longer R25.2
- net at C27.1, C28.1, C30.1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: now also R46.1
- new net: R25.2, R47.1
- no-connect marks 0 -> 1
Other:
- note added: "Rнагр"
