File: Power/fan_555s/fan_555s.kicad_pcb (KiCad board)
At the start: 2 copper layers, 38 x 16 mm, 12 parts, among them J1 Conn_2pin01, J2 Conn_2pin01, T1 1N60G, U1 NE555

Commit message: 2nd
Routing:
- net GND: track 47.5 -> 53.0 mm
- net Net-(U1-CTL): track 3.03 -> 4.87 mm
Changed lines of the file:
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@@
 		(tags "resistor")
 		(property "Reference" "R1"
-			(at 0 1.875 0)
+			(at 0 1.9 0)
 			(layer "F.SilkS")
 			(effects
@@
 		(tags "Through hole pin header THT 1x02 2.54mm single row")
 		(property "Reference" "R2"
-			(at 0.05 -2.405 0)
+			(at -1.725 -2.405 0)
 			(layer "F.SilkS")
 			(effects
@@
 		(tags "capacitor")
 		(property "Reference" "C1"
-			(at -3.22 0 180)
+			(at -3.52 0 180)
 			(layer "F.SilkS")
 			(effects
@@
 		(tags "CMS SOT")
 		(property "Reference" "T1"
-			(at -2 4.63 0)
+			(at 3.55 -3.41 0)
 			(layer "F.SilkS")
 			(effects
@@
 		(tags "D_SOD-123F")
 		(property "Reference" "D1"
-			(at -3.775 0 0)
+			(at -3.775 -0.85 0)
 			(layer "F.SilkS")
 			(effects
@@
 	)
 	(segment
-		(start 52.1 55.05)
-		(end 52.1 52.1)
+		(start 43.8 54.1)
+		(end 43.8 54.4)
 		(width 0.46)
 		(layer "F.Cu")
@@
 	)
 	(segment
-		(start 51.45 55.7)
-		(end 52.1 55.05)
+		(start 43.8 54.9)
+		(end 44.6 55.7)
+		(width 0.46)
+		(layer "F.Cu")
+		(net 2)
+	)
+	(segment
+		(start 46.725 54.2)
+		(end 46.725 55.675)
+		(width 0.46)
+		(layer "F.Cu")
+		(net 2)
+	)
+	(segment
+		(start 46.7 55.7)
+		(end 44.6 55.7)
+		(width 0.46)
+		(layer "F.Cu")
+		(net 2)
+	)
+	(segment
+		(start 44.425 44.875)
+		(end 44.375 44.875)
 		(width 0.46)
 		(layer "F.Cu")
@@
 	(segment
 		(start 43.8 53.2)
-		(end 43.8 45.45)
+		(end 43.8 53)
+		(width 0.46)
+		(layer "F.Cu")
+		(net 2)
+	)
+	(segment
+		(start 52.1 52.1)
+		(end 52.1 55.05)
 		(width 0.46)
 		(layer "F.Cu")
@@
 	)
 	(segment
-		(start 44.8 54.2)
-		(end 43.8 53.2)
-		(width 0.46)
-		(layer "F.Cu")
-		(net 2)
-	)
-	(segment
-		(start 47.2 55.75)
-		(end 47.25 55.7)
+		(start 52.75 51.45)
+		(end 52.1 52.1)
 		(width 0.46)
 		(layer "F.Cu")
@@
 	)
 	(segment
+		(start 44.375 44.875)
+		(end 44.75 44.5)
+		(width 0.46)
+		(layer "F.Cu")
+		(net 2)
+	)
+	(segment
 		(start 59.1 49.77)
 		(end 59.1 51.4)
@@
 	)
 	(segment
-		(start 44.75 44.5)
-		(end 46.198125 44.5)
-		(width 0.46)
-		(layer "F.Cu")
-		(net 2)
-	)
-	(segment
-		(start 46.198125 44.5)
-		(end 47.448125 43.25)
-		(width 0.46)
-		(layer "F.Cu")
-		(net 2)
-	)
-	(segment
-		(start 46.725 55.275)
-		(end 47.2 55.75)
-		(width 0.46)
-		(layer "F.Cu")
-		(net 2)
-	)
-	(segment
-		(start 52.1 52.1)
-		(end 52.75 51.45)
-		(width 0.46)
-		(layer "F.Cu")
-		(net 2)
-	)
-	(segment
-		(start 58.35 51.45)
-		(end 59.15 51.45)
+		(start 51.45 55.7)
+		(end 47.5 55.7)
 		(width 0.46)
 		(layer "F.Cu")
@@
 	(segment
 		(start 46.725 54.2)
-		(end 44.8 54.2)
-		(width 0.46)
-		(layer "F.Cu")
-		(net 2)
-	)
-	(segment
-		(start 52.75 51.45)
-		(end 58.35 51.45)
+		(end 44 54.2)
+		(width 0.46)
+		(layer "F.Cu")
+		(net 2)
+	)
+	(segment
+		(start 46.05 43.25)
+		(end 44.425 44.875)
+		(width 0.46)
+		(layer "F.Cu")
+		(net 2)
+	)
+	(segment
+		(start 47.5 55.7)
+		(end 46.7 55.7)
+		(width 0.46)
+		(layer "F.Cu")
+		(net 2)
+	)
+	(segment
+		(start 46.725 55.675)
+		(end 46.7 55.7)
+		(width 0.46)
+		(layer "F.Cu")
+		(net 2)
+	)
+	(segment
+		(start 43.8 53)
+		(end 43.8 45.45)
+		(width 0.46)
+		(layer "F.Cu")
+		(net 2)
+	)
+	(segment
+		(start 44 54.2)
+		(end 43.8 54.4)
+		(width 0.46)
+		(layer "F.Cu")
+		(net 2)
+	)
+	(segment
+		(start 43.8 54.4)
+		(end 43.8 54.9)
 		(width 0.46)
 		(layer "F.Cu")
@@
 	)
 	(segment
-		(start 47.25 55.7)
-		(end 51.45 55.7)
-		(width 0.46)
-		(layer "F.Cu")
-		(net 2)
-	)
-	(segment
 		(start 43.8 45.45)
-		(end 44.75 44.5)
+		(end 44.375 44.875)
+		(width 0.46)
+		(layer "F.Cu")
+		(net 2)
+	)
+	(segment
+		(start 47.448125 43.25)
+		(end 46.05 43.25)
 		(width 0.46)
 		(layer "F.Cu")
@@
 	)
 	(segment
-		(start 46.725 54.2)
-		(end 46.725 55.275)
-		(width 0.46)
-		(layer "F.Cu")
-		(net 2)
+		(start 52.1 55.05)
+		(end 51.45 55.7)
+		(width 0.46)
+		(layer "F.Cu")
+		(net 2)
+	)
+	(segment
+		(start 59.15 51.45)
+		(end 52.75 51.45)
+		(width 0.46)
+		(layer "F.Cu")
+		(net 2)
+	)
+	(segment
+		(start 43.8 54.1)
+		(end 43.8 53)
+		(width 0.46)
+		(layer "F.Cu")
+		(net 2)
+	)
+	(segment
+		(start 51.15 43.25)
+		(end 50.398125 43.25)
+		(width 0.46)
+		(layer "F.Cu")
+		(net 3)
+	)
+	(segment
+		(start 51.215 46.285)
+		(end 51.5 46)
+		(width 0.46)
+		(layer "F.Cu")
+		(net 3)
+	)
+	(segment
+		(start 51.5 43.6)
+		(end 51.15 43.25)
+		(width 0.46)
+		(layer "F.Cu")
+		(net 3)
 	)
 	(segment
 		(start 50.398125 46.285)
-		(end 50.398125 43.25)
-		(width 0.46)
-		(layer "F.Cu")
+		(end 51.215 46.285)
+		(width 0.46)
+		(layer "F.Cu")
+		(net 3)
+	)
+	(segment
+		(start 51.5 46)
+		(end 51.5 43.6)
+		(width 0.46)
+		(layer "F.Cu")

Commit message: up
Parts:
- H1: footprint MountingHole:MountingHole_3.2mm_M3_DIN965_Pad -> MountingHole:MountingHole_3.2mm_M3
- moved H1 1.10 mm to (76.0, 53.0)
Routing:
- net Net-(D1-C): track 91.7 -> 93.4 mm
- net GND: track 53.0 -> 54.2 mm

Commit message: up
Routing:
- net Net-(D1-A): track 28.7 -> 21.5 mm
Changed lines of the file:
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@@
-	)
-	(segment
-		(start 68.45 47.795)
-		(end 71.6 47.795)
-		(width 0.46)
-		(layer "F.Cu")
-		(net 5)
-	)
-	(segment
-		(start 68.45 47.795)
-		(end 68.45 51.9)
-		(width 0.46)
-		(layer "F.Cu")
-		(net 5)
 	)
 	(segment
