File: Power/fan_555s/fan_555s.kicad_sch (KiCad schematic)
At the start: 12 parts, among them J1 Conn_2pin01, J2 Conn_2pin01, T1 1N60G, U1 NE555

Commit message: up
Parts:
- H1: footprint MountingHole:MountingHole_3.2mm_M3_DIN965_Pad -> MountingHole:MountingHole_3.2mm_M3
Changed lines of the file:
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@@
 			)
 		)
-		(property "Footprint" "MountingHole:MountingHole_3.2mm_M3_DIN965_Pad"
+		(property "Footprint" "MountingHole:MountingHole_3.2mm_M3"
 			(at 105.41 66.04 0)
 			(effects

Commit message: up
Parts:
- D1: value 4148 -> 5819
Changed lines of the file:
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@@
 			)
 		)
-		(property "Value" "4148"
+		(property "Value" "5819"
 			(at 116.84 43.18 0)
 			(effects

Commit message: up
Parts:
- R1: value 22k -> 18k
- R3: value 100 -> 220
