File: Power/psu2psu02/psu2psu02.kicad_pcb (KiCad board)
At the start: 2 copper layers, 126 x 78 mm, 46 parts, among them Q1 740, Q2 740, T1 BC817, T2 BC807, U1 TL494IDR, U2 IR2113S, U3 PC817

Commit message: op
Parts:
- removed D2: ES1J, Diode_SMD:D_SMA
- removed D7: DIODE, Diode_SMD:D_MiniMELF
- removed L1: LFERR, _aTransformers:DRO05-FLEX-200A
- removed R23: 470k, Resistor_SMD:R_1206_3216Metric
- removed R24: 7k5, Resistor_SMD:R_1206_3216Metric
- removed R25, R26: 100k, Resistor_SMD:R_1206_3216Metric
- removed R27: 1k, Resistor_SMD:R_1206_3216Metric
- removed T1: BC817, Package_TO_SOT_SMD:SOT-23
- removed T2: BC807, Package_TO_SOT_SMD:SOT-23
- added C10: 4n7, Capacitor_THT:C_Disc_D4.3mm_W1.9mm_P5.00mm, F.Cu at (139.1, 55.8)
- added C11: 0,1, _aCapa:C_Rect_06-L16P15W5.8, F.Cu at (180.3, 108.7)
- added C18: 1, Capacitor_THT:CP_Radial_D16.0mm_P7.50mm, F.Cu at (163.2, 113.1)
- added C23: 1, Capacitor_THT:CP_Radial_D16.0mm_P7.50mm, F.Cu at (146.6, 113.1)
- added C24: 1, Capacitor_THT:CP_Radial_D16.0mm_P7.50mm, F.Cu at (93.0, 98.8)
- added C9: 0,1, _aCapa:C_Rect_06-L16P15W5.8, F.Cu at (173.0, 82.9)
- added D5: SF10A400H, Package_TO_SOT_THT:TO-220-2_Vertical, F.Cu at (132.3, 91.0)
- added D6: SF10A400H, Package_TO_SOT_THT:TO-220-2_Vertical, F.Cu at (117.0, 91.0)
- added F1: 1A, Fuse:Fuseholder_Clip-5x20mm_Littelfuse_100_Inline_P20.50x4.60mm_D1.30mm_Horizontal, F.Cu at (193.3, 114.7)
- added F3: 3A, Fuse:Fuse_Littelfuse_395Series, F.Cu at (135.8, 54.5)
- added FL1: FEMI-FLEX01, _aTransformers:EMIF02-FLEX, F.Cu at (177.8, 95.8)
- added J3: Conn_2pin01, Connector_Phoenix_GMSTB:PhoenixContact_GMSTBVA_2,5_2-G-7,62_1x02_P7.62mm_Vertical, F.Cu at (201.9, 97.8)
- added J6: ACDC_China-01, _aModules:ACDC_China-04, F.Cu at (165.7, 48.5)
- added R11: 07K180, Varistor:RV_Disc_D12mm_W3.9mm_P7.5mm, F.Cu at (188.0, 95.4)
- added R28: 3k, _aResistors:RES2WV01, F.Cu at (144.6, 49.3)
- added R50: t°, Varistor:RV_Disc_D12mm_W3.9mm_P7.5mm, F.Cu at (194.3, 105.3)
- added TV1: TV, _aTransformers:DRO05-FLEX-200A, F.Cu at (112.7, 80.2)
- C17, C22: footprint Capacitor_THT:CP_Radial_D18.0mm_P7.50mm -> Capacitor_THT:CP_Radial_D22.0mm_P10.00mm_SnapIn
- C20: value 100x35 -> 1; footprint Capacitor_THT:CP_Radial_D6.3mm_P2.50mm -> Capacitor_THT:CP_Radial_D16.0mm_P7.50mm
- D3: value ES1J -> SF10A400H; footprint Diode_SMD:D_SMA -> Package_TO_SOT_THT:TO-220-2_Vertical
- D4: value ~ -> SF10A400H; footprint Package_TO_SOT_THT:TO-220-3_Vertical -> Package_TO_SOT_THT:TO-220-2_Vertical
- moved C20 71.5 mm to (93.0, 81.2), turned to 180 degrees
- moved HS2 53.5 mm to (127.4, 44.0)
- moved HS1 51.8 mm to (134.2, 96.2)
- moved D3 40.1 mm to (165.7, 91.0), turned to 180 degrees
- moved C17 39.6 mm to (194.7, 54.8), turned to -90 degrees
- moved C22 31.8 mm to (194.7, 77.3), turned to -90 degrees
- moved Q1 11.8 mm to (133.2, 49.3)
- moved R9 9.92 mm to (128.4, 49.3)
- moved R5 9.52 mm to (113.0, 61.9)
- moved R6 9.52 mm to (110.7, 61.9)
- moved TR1 8.40 mm to (147.1, 71.3)
- moved RS1 8.13 mm to (180.4, 77.7)
- moved C7 7.94 mm to (177.8, 59.0)
- moved C8 7.94 mm to (167.9, 74.0)
- moved C19 7.73 mm to (109.3, 56.5)
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Connections:
- net Net-(C7-Pad1) renamed /HV6
- net Net-(Q1-S) renamed /HV4
- C20 pad 1: Net-(D2-C) -> Net-(C20-Pad1)
- C20 pad 2: GND2 -> GND
- D3 pad 1: Net-(D2-C) -> Net-(D3-C)
- D4 pad 1: Net-(D4-A1) -> Net-(D3-A)
- Q1 pad 2: +HV -> Net-(Q1-D)
- RS1 pad 2: unconnected-(RS1-Pad2) -> Net-(C9-Pad2)
- RS1 pad 3: unconnected-(RS1-Pad3) -> Net-(C9-Pad1)
- TR1 pad 1: Net-(D2-A) -> unconnected-(TR1-Pad1)
- TR1 pad 11: Net-(D4-A2) -> Net-(D3-A)
- TR1 pad 12: Net-(D4-A2) -> Net-(D3-A)
- TR1 pad 2: Net-(D3-A) -> unconnected-(TR1-Pad2)
- TR1 pad 7: Net-(D4-A1) -> Net-(D5-A)
- TR1 pad 8: Net-(D4-A1) -> Net-(D5-A)
Routing:
- net GND: track 0.00 -> 154.8 mm, vias 0 -> 2
- net Net-(C18-Pad2): track 0.00 -> 107.3 mm
- net Net-(D3-C): track 0.00 -> 70.6 mm
- net Net-(C9-Pad1): track 0.00 -> 63.3 mm
- net Net-(C9-Pad2): track 0.00 -> 58.5 mm
- net Net-(F1-Pad1): track 0.00 -> 42.0 mm
- net Net-(D5-A): track 0.00 -> 39.2 mm
- net Net-(C20-Pad1): track 0.00 -> 38.1 mm
- net Net-(C11-Pad1): track 0.00 -> 35.9 mm
- net Net-(C11-Pad2): track 0.00 -> 27.0 mm
- net Net-(J3-Pad1): track 0.00 -> 22.1 mm
- net Net-(D2-C): track 21.4 -> 0.00 mm
- net +HV: track 80.2 -> 100.4 mm, vias 1 -> 0
- net Net-(D7-A): track 19.2 -> 0.00 mm
- net Net-(D3-A): track 4.47 -> 23.0 mm
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
Commit message: up
Routing:
- net Net-(D3-C): track 70.6 -> 26.4 mm
Changed lines of the file:
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@@
-	)
-	(segment
-		(start 162.775 86.775)
-		(end 162.775 79.3)
-		(width 2)
-		(layer "B.Cu")
-		(net 43)
-	)
-	(segment
-		(start 162.125 78.65)
-		(end 131.8 78.65)
-		(width 2)
-		(layer "B.Cu")
-		(net 43)
 	)
 	(segment
 		(start 132.265 88.64)
 		(end 132.265 90.975)
-		(width 2)
-		(layer "B.Cu")
-		(net 43)
-	)
-	(segment
-		(start 162.775 79.3)
-		(end 162.125 78.65)
 		(width 2)
 		(layer "B.Cu")
@@
 	)
 	(segment
-		(start 165.74 90.975)
-		(end 165.74 89.74)
-		(width 2)
-		(layer "B.Cu")
-		(net 43)
-	)
-	(segment
 		(start 130.775 87.15)
 		(end 132.265 88.64)
 		(width 2)
 		(layer "B.Cu")
-		(net 43)
-	)
-	(segment
-		(start 165.74 89.74)
-		(end 162.775 86.775)
-		(width 2)
-		(layer "B.Cu")
